Commit message: add two break beams in launch; cleanup prox ray plugins

File: models/break_beam/break_beam.gazebo.xacro (robot description, xacro)
@@ -33,6 +33,4 @@
         <always_on>1</always_on>
         <plugin name="${prefix}controller" filename="libROSProximityRayPlugin.so" >
-          <topicName>laser/scan</topicName>
-          <frameName>${prefix}optical_link</frameName>
         </plugin>
       </sensor>

File: models/break_beam/break_beam.urdf.xacro (robot description, xacro)
@@ -34,5 +34,5 @@
       <parent link="${prefix}world_interface" />
       <child link="${prefix}base_link" />
-      <origin xyz="1.6 2.7 0.925" rpy="0 0 ${radians(180)}" />
+      <origin xyz="0 0 0" rpy="0 0 ${radians(180)}" />
     </joint>
     <joint name="${prefix}joint_1" type="fixed">
