Commit message: added vacuum gripper

File: models/ur5/ur5.urdf.xacro (robot description, xacro)
@@ -330,4 +330,34 @@
       </collision>
     </link>
+    <link name="left_end_effector">
+      <gravity>0</gravity>
+      <visual>
+        <origin rpy="0 0 0" xyz="0 0 0"/>
+        <geometry>
+          <box size="0.01 0.01 0.01"/>
+        </geometry>
+        <material name="transparent">
+          <color rgba="0 0 0 0"/>
+        </material>
+      </visual>
+      <inertial>
+        <origin rpy="0 0 0" xyz="0.000000 0.000000 0.000000"/>
+        <mass value="0.0001"/>
+        <inertia ixx="1e-08" ixy="0" ixz="0" iyy="1e-08" iyz="0" izz="1e-08"/>
+      </inertial>
+    </link>
+    <joint name="left_end_joint" type="revolute">
+      <parent link="wrist_3_link" />
+      <child link="left_end_effector" />
+      <origin rpy="0 0 0" xyz="0.08 0 .44" />
+      <limit effort="30" velocity="1.0" lower="0" upper="0" />
+    </joint>
+    <gazebo>
+      <plugin name="gazebo_ros_vacuum_gripper" filename="libgazebo_ros_vacuum_gripper.so">
+        <robotNamespace>/robot/left_vacuum_gripper</robotNamespace>
+        <bodyName>left_end_effector</bodyName>
+        <topicName>grasping</topicName>
+      </plugin>
+    </gazebo>
     <xacro:ur_arm_transmission prefix="${prefix}" hw_interface="${transmission_hw_interface}" />
     <xacro:ur_arm_gazebo prefix="${prefix}" />

File: models/ur5/ur5_robot.urdf.xacro (robot description, xacro)
@@ -11,4 +11,8 @@
     transmission_hw_interface="$(arg transmission_hw_interface)"
   />
+  <!-- vacuum gripper -->
+  <xacro:property name="simple_gripper" value="simple_gripper_" />
+  <xacro:include filename="$(find ur5_t2_4230)/urdf/simple_gripper/simple_gripper.xacro"/>
+  <xacro:simple_gripper prefix="simple_gripper_"/>
   <link name="world" />
   <joint name="world_joint" type="fixed">
@@ -17,3 +21,15 @@
     <origin xyz="0.0 0.0 0.0" rpy="0.0 0.0 0.0" />
   </joint>
+  <!-- Simple Vacuum Gripper -->
+  <xacro:include filename="$(find ur5_t2_4230)/urdf/simple_gripper/simple_gripper.urdf.xacro"/>
+  <xacro:simple_gripper_urdf prefix="${simple_gripper_prefix}"/>
+  <xacro:include filename="$(find ur5_t2_4230)/urdf/simple_gripper/simple_gripper.gazebo.xacro"/>
+  <xacro:simple_gripper_gazebo prefix="${simple_gripper_prefix}" gripper_link="robot_system_::robot_wrist_3_link">
+    <drops_info/>
+  </xacro:simple_gripper_gazebo>
+  <!-- Joints -->
+  <joint name="gripper_to_robot" type="fixed">
+    <parent link="${robot_prefix}tool0" />
+    <child link="${simple_gripper_prefix}base_link" />
+  </joint>
 </robot>

Commit message: progress on vacuum gripper; turn on debugging variables (todo: cleanup)

File: models/ur5/ur5.urdf.xacro (robot description, xacro)
@@ -335,5 +335,5 @@
         <origin rpy="0 0 0" xyz="0 0 0"/>
         <geometry>
-          <box size="0.01 0.01 0.01"/>
+          <box size="0.05 0.05 0.05"/>
         </geometry>
         <material name="transparent">
@@ -350,12 +350,25 @@
       <parent link="wrist_3_link" />
       <child link="left_end_effector" />
-      <origin rpy="0 0 0" xyz="0.08 0 .44" />
+      <origin rpy="0 0 0" xyz="0.00 0.07 0.00" />
       <limit effort="30" velocity="1.0" lower="0" upper="0" />
     </joint>
     <gazebo>
-      <plugin name="gazebo_ros_vacuum_gripper" filename="libgazebo_ros_vacuum_gripper.so">
+      <!-- <plugin name="gazebo_ros_vacuum_gripper" filename="libgazebo_ros_vacuum_gripper.so">
         <robotNamespace>/robot/left_vacuum_gripper</robotNamespace>
         <bodyName>left_end_effector</bodyName>
-        <topicName>grasping</topicName>
+        <topicName>enable</topicName>
+      </plugin> -->
+      <plugin name="ros_vacuum_gripper" filename="libROSVacuumGripperPlugin.so">
+        <grasp_check>
+          <detach_steps>40</detach_steps>
+          <attach_steps>1</attach_steps>
+          <min_contact_count>1</min_contact_count>
+        </grasp_check>
+        <!-- <xacro:insert_block name="drops_info" /> -->
+        <suction_cup_link>left_end_effector</suction_cup_link>
+        <!-- ROS -->
+        <robot_namespace>/robot/left_vacuum_gripper</robot_namespace>
+        <control_topic>gripper/control</control_topic>
+        <state_topic>gripper/state</state_topic>
       </plugin>
     </gazebo>

File: models/ur5/ur5_robot.urdf.xacro (robot description, xacro)
@@ -23,13 +23,13 @@
   <!-- Simple Vacuum Gripper -->
   <xacro:include filename="$(find ur5_t2_4230)/urdf/simple_gripper/simple_gripper.urdf.xacro"/>
-  <xacro:simple_gripper_urdf prefix="${simple_gripper_prefix}"/>
+  <xacro:simple_gripper_urdf prefix="simple_gripper_"/>
   <xacro:include filename="$(find ur5_t2_4230)/urdf/simple_gripper/simple_gripper.gazebo.xacro"/>
-  <xacro:simple_gripper_gazebo prefix="${simple_gripper_prefix}" gripper_link="robot_system_::robot_wrist_3_link">
+  <xacro:simple_gripper_gazebo prefix="simple_gripper_" gripper_link="wrist_3_link">
     <drops_info/>
   </xacro:simple_gripper_gazebo>
   <!-- Joints -->
   <joint name="gripper_to_robot" type="fixed">
-    <parent link="${robot_prefix}tool0" />
-    <child link="${simple_gripper_prefix}base_link" />
+    <parent link="tool0" />
+    <child link="simple_gripper_base_link" />
   </joint>
 </robot>

File: urdf/simple_gripper/simple_gripper.gazebo.xacro (robot description, xacro)
@@ -15,5 +15,5 @@
           <min_contact_count>1</min_contact_count>
         </grasp_check>
-        <xacro:insert_block name="drops_info" />
+        <drops_info/>
         <suction_cup_link>${gripper_link}</suction_cup_link>
         <!-- ROS -->

Commit message: implement functional vacuum gripper; change robot movement on pickup object

File: models/ur5/ur5.urdf.xacro (robot description, xacro)
@@ -332,12 +332,15 @@
     <link name="left_end_effector">
       <gravity>0</gravity>
-      <visual>
+      <collision name="collision">
         <origin rpy="0 0 0" xyz="0 0 0"/>
         <geometry>
-          <box size="0.05 0.05 0.05"/>
-        </geometry>
-        <material name="transparent">
-          <color rgba="0 0 0 0"/>
-        </material>
+          <cylinder length="0.005" radius="0.02"/>
+        </geometry>
+      </collision>
+      <visual>
+        <origin rpy="0 0 0" xyz="0 0 0"/>
+        <geometry>
+          <cylinder length="0.005" radius="0.02"/>
+        </geometry>
       </visual>
       <inertial>
@@ -350,5 +353,5 @@
       <parent link="wrist_3_link" />
       <child link="left_end_effector" />
-      <origin rpy="0 0 0" xyz="0.00 0.07 0.00" />
+      <origin rpy="${pi/2} 0 0" xyz="0.00 0.085 0.00" />
       <limit effort="30" velocity="1.0" lower="0" upper="0" />
     </joint>
@@ -365,5 +368,4 @@
           <min_contact_count>1</min_contact_count>
         </grasp_check>
-        <!-- <xacro:insert_block name="drops_info" /> -->
         <suction_cup_link>left_end_effector</suction_cup_link>
         <!-- ROS -->
